File: 05-am-radio/schematics/am-radio.kicad_sch (KiCad schematic)
At the start: 0 parts

Commit message: schem almost doner
Parts:
- added C1, C2, C3, C5, C9: 0.1u, symbol Device:C_Small
- added C4, C8: 10n, symbol Device:C_Small
- added C6, C7: 1n, symbol Device:C_Small
- added D1, D2, D3: 1N5819, Diode_THT:D_DO-41_SOD81_P10.16mm_Horizontal, symbol Diode:1N5819
- added J1, J2: AudioJack2_Ground, symbol Connector_Audio:AudioJack2_Ground
- added R1, R10, R11, R12, R2, R3, R4, R6, R7, R8: 1k, symbol Device:R_US
- added R13, R14: 1.2k, symbol Device:R_US
- added R15: 8.2k, symbol Device:R_US
- added R16: 2.7k, symbol Device:R_US
- added R17, R18: 33k, symbol Device:R_US
- added R5, R9: 150, symbol Device:R_US
- added RV1, RV3: 10k, symbol Device:R_Potentiometer_US
- added RV2: 100k, symbol Device:R_Potentiometer_US
- added U1: LM324, symbol Amplifier_Operational:LM324
- added U2, U3, U6: AD633JRZ-R7, AD633JRZ-R7:SOIC127P600X175-8N, symbol AD633JRZ-R7:AD633JRZ-R7
- added U4, U7, U8: LF356, symbol Amplifier_Operational:LF356
- added U5: LMC555xM, Package_SO:SOIC-8_3.9x4.9mm_P1.27mm, symbol Timer:LMC555xM
Connections:
- new net: RV1.2, U1.10 (+)
- new net: C6.2, R17.2, U7.2 (-)
- new net: C7.1, R17.1, U7.6, U8.3 (+)
- new net: C8.1, C9.1, D3.1 (K), R18.1
- new net: J2.S, R3.1
- new net: R3.2, R4.2, R9.1
- new net: J2.T, R4.1
- new net: C6.1, C7.2, R15.2, R16.1
- new net: R5.2, R6.2, R7.1, U1.2 (-)
- new net: D1.1 (K), D2.2 (A), RV3.1
- new net: C4.1, RV3.2, U5.2 (TR), U5.6 (THR)
- new net: D1.2 (A), R13.2, R14.1, U5.7 (DIS)
- new net: D2.1 (K), R14.2
- new net: J1.S, R1.1
- new net: R1.2, R2.2, R5.1
- new net: R11.2, R12.2, RV2.3, U4.2 (-)
- new net: J1.T, R2.1
- new net: C3.1, U5.5 (CV)
- new net: R10.1, R8.2, R9.2, U1.6 (-)
- new net: C5.1, U5.3 (Q)
- new net +10V: C1.1, R13.1, RV1.1, U1.4 (V+), U2.6 (+VS), U3.6 (+VS), U4.7 (V+), U5.4 (R), U5.8 (VCC), U6.6 (+VS), U7.7 (V+), U8.7 (V+)
- new net -10V: C2.1, U1.11 (V-), U2.3 (-VS), U3.3 (-VS), U4.4 (V-), U6.3 (-VS), U7.4 (V-), U8.4 (V-)
- new net GND: C1.2, C2.2, C3.2, C4.2, C8.2, J1.G, J2.G, R16.2, R18.2, RV1.3, U1.3 (+), U1.5 (+), U2.2 (Y2), U2.4 (Z), U2.8 (X2), U3.2 (Y2), U3.4 (Z), U3.8 (X2), U4.3 (+), U5.1 (GND), U6.2 (Y2), U6.4 (Z), U6.8 (X2), U7.3 (+)
- new net VIF: R15.1, U6.5 (W)
- new net VLO: C5.2, U6.1 (Y1)
- new net V_m1: R7.2, U1.1
- new net V_m2: R10.2, U1.7
- new net V_offset: R6.1, R8.1, U1.8, U1.9 (-)
- new net Vam: RV2.2, U4.6, U6.7 (X1)
- new net Vcarrier1: U2.1 (Y1)
- new net Vcarrier2: U3.1 (Y1)
- new net Vfilt: U8.2 (-), U8.6
- new net Vm1: U2.7 (X1)
- new net Vm2: U3.7 (X1)
- new net Vmodulated1: R12.1, U2.5 (W)
- new net Vmodulated2: R11.1, U3.5 (W)
- no-connect marks 0 -> 9
Other:
- note added: "10kHz Band Pass Filter"
- note added: "AM Generation"
- note added: "AM Mixing & Summing"
- note added: "Adjustable Frequency wave for demodulation"
- note added: "Demodulation"
- note added: "Filtering & Amplification"
- note added: "Final modulated signal with 2 stations"
- note added: "From Wavegen"
- note added: "Generating Input Messages"
- note added: "Superhet Receiver"
- note added: "Vam demodulated to an intermediate frequency 10kHz."
- note added: "Vm1 = A(1 + m*x1(t))"
- note added: "Vm2 = A(1 + m*x2(t))"

Commit message: schem done
Parts:
- added C10: 0.05u, symbol Device:C_Small
- added LS1: Speaker, symbol Device:Speaker
- added R19: 10, symbol Device:R_US
- added U9: LM386, symbol Amplifier_Audio:LM386
Connections:
- net +10V: now also U9.6 (V+)
- net GND: now also LS1.2, R19.2, U9.2 (-), U9.4 (GND)
- net Vfilt: now also D3.2 (A)
- net Vfinal: now reaches C9.2
- net Vfinal: now also U9.3 (+)
- new net: C10.2, R19.1
- new net: C10.1, LS1.1, U9.5
- no-connect marks 9 -> 12
Other:
- note added: "Audio Amplifier"
- note added: "Envelope Detector"
- moved on the sheet: C8, C9, D3, R18
